File: media/week11/eagle/tiny44/tiny44.sch (EAGLE design)
At the start: 10 parts, among them IC1 ATTINY44-SSU, X1 22-23-2041, X3 22-23-2041

Commit message: week11 and start week16
Parts:
- removed X1, X3: 22-23-2041, con-molex:22-23-2041
- added X2, X4: (no value), con-molex:KK-156-7
Connections:
- removed net N$10: IC1.(PCINT2/AIN1/ADC2)PA2
- removed net N$2: IC1.(PCINT10/INT0/OC0A/CKOUT)PB2
- removed net N$3: IC1.(PCINT9/XTAL2)PB1, U$1.3
- removed net N$4: IC1.(PCINT8/XTAL1/CLKI)PB0, U$1.1
- removed net N$5: IC1.(PCINT7/ICP/OC0B/ADC7)PA7
- removed net N$9: IC1.(PCINT3/T0/ADC3)PA3
- removed net PT1: X3-3.S
- removed net PT2: X3-2.S
- new net 10: IC1.(PCINT8/XTAL1/CLKI)PB0, U$1.1, X4-6.S
- new net 8: IC1.(PCINT10/INT0/OC0A/CKOUT)PB2, X4-3.S
- new net 9: IC1.(PCINT9/XTAL2)PB1, U$1.3, X4-5.S
- new net A2: IC1.(PCINT2/AIN1/ADC2)PA2, X2-4.S
- new net A3: IC1.(PCINT3/T0/ADC3)PA3, X2-5.S
- new net A7: IC1.(PCINT7/ICP/OC0B/ADC7)PA7, X4-2.S
- net GND: now also X2-1.S; no longer X3-4.S
- net MISO: now also X2-7.S; no longer X1-3.S
- net MOSI: now also X4-1.S; no longer X1-4.S
- net RST: now also X4-4.S; no longer X3-1.S
- net RX: now also X2-3.S
- net SCK: now also X2-6.S; no longer X1-2.S
- net TX: now also X2-2.S
- net VCC: now also X4-7.S; no longer X1-1.S
Other:
- moved on the sheet: R4, U$6
